Commit message: modells updated with namespace

File: realsense2_description/urdf/_d415.urdf.xacro (robot description, xacro)
@@ -19,13 +19,9 @@
 aluminum peripherial evaluation case.
 -->
-<robot name="sensor_d415" xmlns:xacro="http://ros.org/wiki/xacro"
-       xmlns:nw="urn:template:template-network"
-       xmlns:nt="urn:template:template-network-topology"
-       xmlns:l1t="urn:template:template-l1"
-       xmlns:l2t="urn:template:template-l2">
+<robot name="sensor_d415" xmlns:xacro="http://ros.org/wiki/xacro">
   <!-- Includes -->
   <xacro:include filename="$(find realsense2_description)/urdf/_materials.urdf.xacro" />
   <xacro:include filename="$(find realsense2_description)/urdf/_usb_plug.urdf.xacro" />
-  <xacro:include filename="$(find interface-description)/urdf/usb30.urdf.xacro" />
+  <!-- <xacro:include filename="$(find interface-description)/urdf/usb30.urdf.xacro" /> -->
   <xacro:macro name="sensor_d415" params="parent *origin  name:=camera  use_nominal_extrinsics:=false add_plug:=false use_mesh:=true">
     <xacro:property name="M_PI" value="3.1415926535897931" />
@@ -148,39 +144,4 @@
       </xacro:usb_plug>
     </xacro:if>
-    <yang>
-      <!-- L2 network topology -->
-      <nw:network>
-        <nw:network-id>${L2_network_id}</nw:network-id>
-        <nw:network-types>
-          <l2t:l2-topology/>
-        </nw:network-types>
-        <nw:supporting-network>
-          <nw:network-ref>${L1_network_id}</nw:network-ref>
-        </nw:supporting-network>
-        <nw:node>
-          <nw:node-id>${L2_id}</nw:node-id>
-          <nw:supporting-node>
-            <nw:network-ref>${L1_network_id}</nw:network-ref>
-            <nw:node-ref>${L1_id}</nw:node-ref>
-          </nw:supporting-node>
-          <xacro:usb30_L2 id="usb_1" supporting_network="${L1_network_id}" supporting_node="${L1_id}" supporting_tp="usb_1"/>
-        </nw:node>
-      </nw:network>
-      <!-- Physical network topology -->
-      <nw:network>
-        <nw:network-id>${L1_network_id}</nw:network-id>
-        <nw:network-types>
-          <l1t:l1-topology/>
-        </nw:network-types>
-        <nw:node>
-          <nw:node-id>${L1_id}</nw:node-id>
-          <l1t:l1-node-attributes>
-            <l1t:device-type>camera</l1t:device-type>
-          </l1t:l1-node-attributes>
-          <xacro:usb30_L1 id="usb_1"/>
-        </nw:node>
-      </nw:network>
-    </yang>
-  </xacro:macro>
   </xacro:macro>
 </robot>

File: realsense2_description/urdf/_d455.urdf.xacro (robot description, xacro)
@@ -185,5 +185,4 @@
     </xacro:if>
     <yang>
-      <!-- L2 network topology -->
       <xacro:macro name="usb30_L2" params="L1_id:=alma L2_id:=barack L1_network_id:=citrom L2_network_id:=dinnye">
         <nw:network>
