Commit message: redefine macros for interfaces

File: realsense2_description/urdf/_d455.urdf.xacro (robot description, xacro)
@@ -19,7 +19,7 @@
 aluminum peripherial evaluation case.
 -->
-<robot name="sensor_d455" xmlns:xacro="http://ros.org/wiki/xacro"
-       xmlns:nw="urn:template-network"
-       xmlns:nt="urn:network-topology"
+<robot name="sensor_d455"
+       xmlns:xacro="http://ros.org/wiki/xacro"
+       xmlns:nw="urn:network"
        xmlns:l1t="urn:layer1"
        xmlns:l2t="urn:layer2">
@@ -27,5 +27,5 @@
   <xacro:include filename="$(find realsense2_description)/urdf/_materials.urdf.xacro" />
   <xacro:include filename="$(find realsense2_description)/urdf/_usb_plug.urdf.xacro" />
-  <xacro:macro name="sensor_d455" params="parent *origin name:=camera use_nominal_extrinsics:=false L1_id L2_id L1_network_id L2_network_id">
+  <xacro:macro name="sensor_d455" params="parent *origin name:=camera use_nominal_extrinsics:=false">
     <xacro:arg name="add_plug" default="false" />
     <xacro:property name="M_PI" value="3.1415926535897931" />
@@ -186,35 +186,33 @@
     <yang>
       <!-- L2 network topology -->
-      <nw:network>
-        <nw:network-id>${L2_network_id}</nw:network-id>
-        <nw:network-types>
-          <l2t:l2-topology/>
-        </nw:network-types>
-        <nw:supporting-network>
-          <nw:network-ref>${L1_network_id}</nw:network-ref>
-        </nw:supporting-network>
-        <nw:node>
-          <nw:node-id>${L2_id}</nw:node-id>
-          <nw:supporting-node>
-            <nw:network-ref>${L1_network_id}</nw:network-ref>
-            <nw:node-ref>${L1_id}</nw:node-ref>
-          </nw:supporting-node>
-          <xacro:usb30_L2 id="usb_1" supporting_network="${L1_network_id}" supporting_node="${L1_id}" supporting_tp="usb_1"/>
-        </nw:node>
-      </nw:network>
-      <!-- Physical network topology -->
-      <nw:network>
-        <nw:network-id>${L1_network_id}</nw:network-id>
-        <nw:network-types>
-          <l1t:l1-topology/>
-        </nw:network-types>
-        <nw:node>
-          <nw:node-id>${L1_id}</nw:node-id>
-          <l1t:l1-node-attributes>
-            <l1t:device-type>camera</l1t:device-type>
-          </l1t:l1-node-attributes>
-          <xacro:usb30_L1 id="usb_1"/>
-        </nw:node>
-      </nw:network>
+      <xacro:macro name="usb30_L2" params="L1_id:=alma L2_id:=barack L1_network_id:=citrom L2_network_id:=dinnye">
+        <nw:network>
+          <nw:network-id name="${L2_network_id}"/>
+          <nw:network-types>
+            <l2t:l2-topology/>
+          </nw:network-types>
+          <nw:supporting-network>
+            <nw:network-ref name="${L1_network_id}"/>
+          </nw:supporting-network>
+          <nw:node>
+            <nw:node-id name="${L2_id}"/>
+            <nw:supporting-node>
+              <nw:network-ref name="${L1_network_id}"/>
+              <nw:node-ref name="${L1_id}"/>
+            </nw:supporting-node>
+            <xacro:usb30_L2 id="usb_1" supporting_network="${L1_network_id}" supporting_node="${L1_id}" supporting_tp="usb_1"/>
+          </nw:node>
+          <nw:network-id name="${L1_network_id}"/>
+          <nw:network-types>
+            <l1t:l1-topology/>
+          </nw:network-types>
+          <nw:node id="${L1_id}">
+            <l1t:l1-node-attributes>
+              <l1t:device-type name="camera"/>
+            </l1t:l1-node-attributes>
+            <xacro:usb30_L1 id="usb_1"/>
+          </nw:node>
+        </nw:network>
+      </xacro:macro>
     </yang>
   </xacro:macro>

Commit message: ros layer added

File: realsense2_description/urdf/_d455.urdf.xacro (robot description, xacro)
@@ -185,5 +185,5 @@
     </xacro:if>
     <yang>
-      <xacro:macro name="usb30_L2" params="L1_id:=alma L2_id:=barack L1_network_id:=citrom L2_network_id:=dinnye">
+      <xacro:macro name="sensor_d455" params="L2_network_id:=Data_Link L1_network_id:=Physical L2_id:=d455_Cam_L2 L1_id:=d455_Cam_L1 L3_network_id:=d455_Cam_ROS L3_id:=realsense2_camera">
         <nw:network>
           <nw:network-id name="${L2_network_id}"/>
@@ -212,4 +212,106 @@
             <xacro:usb30_L1 id="usb_1"/>
           </nw:node>
+          <!-- ROS node graph -->
+          <nw:network-id name="${L3_network_id}"/>
+          <nw:network-types>
+            <ros:ros-node-graph/>
+          </nw:network-types>
+          <nw:supporting-network>
+            <nw:network-ref name="${L2_network_id}"/>
+          </nw:supporting-network>
+          <!-- publishes to -->
+          <nt:link>
+            <nt:link-id name="camera_publisher"/>
+            <nt:source>
+              <nt:source-node name="realsense2_camera"/>
+              <nt:source-tp>pub</nt:source-tp>
+            </nt:source>
+            <nt:destination>
+              <nt:dest-node>img_proc</nt:dest-node>
+              <nt:dest-tp>pub</nt:dest-tp>
+            </nt:destination>
+          </nt:link>
+           <!-- publishes to -->
+          <nt:link>
+            <nt:link-id name="model_node"/>
+            <nt:source>
+              <nt:source-node name="robot_state_publisher"/>
+              <nt:source-tp>pub</nt:source-tp>
+            </nt:source>
+            <nt:destination>
+              <nt:dest-node>transform</nt:dest-node>
+              <nt:dest-tp>pub</nt:dest-tp>
+            </nt:destination>
+          </nt:link>
+          <!-- color image topic -->
+          <nw:node>
+            <nw:node-id name="/camera/camera/color/camera_raw"/>
+            <ros:ros-node-attributes>
+              <ros:ros-node-type name=>topic</ros:ros-node-type>
+              <ros:topic-type name="sensor_msgs/msg/Image"/>
+            </ros:ros-node-attributes>
+            <nt:termination-point>
+              <nt:tp-id>pub</nt:tp-id>
+            </nt:termination-point>
+            <nt:termination-point>
+              <nt:tp-id>sub</nt:tp-id>
+            </nt:termination-point>
+          </nw:node>
+          <!-- color camera info topic -->
+          <nw:node>
+            <nw:node-id name="/camera/camera/color/camera_info"/>
+            <ros:ros-node-attributes>
+              <ros:ros-node-type name=>topic</ros:ros-node-type>
+              <ros:topic-type name="sensor_msgs/msg/CameraInfo"/>
+            </ros:ros-node-attributes>
+            <nt:termination-point>
+              <nt:tp-id>pub</nt:tp-id>
+            </nt:termination-point>
+            <nt:termination-point>
+              <nt:tp-id>sub</nt:tp-id>
+            </nt:termination-point>
+          </nw:node>
+          <!-- depth image topic -->
+          <nw:node>
+            <nw:node-id name="/camera/camera/aligned_depth_to_color/image_raw"/>
+            <ros:ros-node-attributes>
+              <ros:ros-node-type name=>topic</ros:ros-node-type>
+              <ros:topic-type name="sensor_msgs/msg/Image"/>
+            </ros:ros-node-attributes>
+            <nt:termination-point>
+              <nt:tp-id>pub</nt:tp-id>
+            </nt:termination-point>
+            <nt:termination-point>
+              <nt:tp-id>sub</nt:tp-id>
+            </nt:termination-point>
+          </nw:node>
+          <!-- depth camera info topic -->
+          <nw:node>
+            <nw:node-id name="/camera/camera/depth/camera_info"/>
+            <ros:ros-node-attributes>
+              <ros:ros-node-type name=>topic</ros:ros-node-type>
+              <ros:topic-type name="sensor_msgs/msg/CameraInfo"/>
+            </ros:ros-node-attributes>
+            <nt:termination-point>
+              <nt:tp-id>pub</nt:tp-id>
+            </nt:termination-point>
+            <nt:termination-point>
+              <nt:tp-id>sub</nt:tp-id>
+            </nt:termination-point>
+          </nw:node>
+          <!-- TF topic -->
+          <nw:node>
+            <nw:node-id name="tf_static"/>
+            <ros:ros-node-attributes>
+              <ros:ros-node-type>topic</ros:ros-node-type>
+              <ros:topic-type name="tf2_msgs/msg/TFMessage"/>
+            </ros:ros-node-attributes>
+            <nt:termination-point>
+              <nt:tp-id>pub</nt:tp-id>
+            </nt:termination-point>
+            <nt:termination-point>
+              <nt:tp-id>sub</nt:tp-id>
+            </nt:termination-point>
+          </nw:node>
         </nw:network>
       </xacro:macro>

Commit message: Fixed camera yang.

File: realsense2_description/urdf/_d455.urdf.xacro (robot description, xacro)
@@ -187,76 +187,85 @@
     </xacro:if>
     <yang>
-      <xacro:macro name="sensor_d455" params="L2_network_id:=Data_Link L1_network_id:=Physical L2_id:=d455_Cam_L2 L1_id:=d455_Cam_L1 L3_network_id:=d455_Cam_ROS L3_id:=realsense2_camera">
-          <nw:network-id name="${L2_network_id}"/>
-          <nw:network-types>
-            <l2t:l2-topology/>
-          </nw:network-types>
-          <nw:supporting-network>
-            <nw:network-ref name="${L1_network_id}"/>
-          </nw:supporting-network>
-          <nw:node>
-            <nw:node-id name="${L2_id}"/>
-            <nw:supporting-node>
-              <nw:network-ref name="${L1_network_id}"/>
-              <nw:node-ref name="${L1_id}"/>
-            </nw:supporting-node>
-            <xacro:usb30_L2 id="usb_1" supporting_network="${L1_network_id}" supporting_node="${L1_id}" supporting_tp="usb_1"/>
-          </nw:node>
-          <nw:network-id name="${L1_network_id}"/>
-          <nw:network-types>
-            <l1t:l1-topology/>
-          </nw:network-types>
-          <nw:node id="${L1_id}">
-            <l1t:l1-node-attributes>
-              <l1t:device-type name="camera"/>
-            </l1t:l1-node-attributes>
-            <xacro:usb30_L1 id="usb_1"/>
-          </nw:node>
-          <nw:network-id name="ros"/>
-          <nw:network-types>
-            <ros:ros-node-graph/>
-          </nw:network-types>
-          <nw:supporting-network>
-            <nw:network-ref name="${L2_network_id}"/>
-          </nw:supporting-network>
-          <nw:node> <!-- /camera/realsense2_camera ROS node -->
-            <nw:node-id name="realsense2-camera" /> <!--(node-name)-->
-            <ros:ros-node-attributes>
-              <ros:ros-node-type>node</ros:ros-node-type>
-            </ros:ros-node-attributes>
-            <nt:termination-point>
-              <nt:tp-id>pub</nt:tp-id>
-            </nt:termination-point>
-            <nt:termination-point>
-              <nt:tp-id>sub</nt:tp-id>
-            </nt:termination-point>
-          </nw:node>
-          <nw:node> <!-- /tf_static topic -->
-            <nw:node-id name="/camera/color/image_raw" />
-            <ros:ros-node-attributes>
-              <ros:ros-node-type>topic</ros:ros-node-type>
-              <ros:topic-type name="sensor_msgs/msg/Image" hz="30" bw="83.34MB/s"/>
-            </ros:ros-node-attributes>
-            <nt:termination-point>
-              <nt:tp-id>pub</nt:tp-id>
-            </nt:termination-point>
-            <nt:termination-point>
-              <nt:tp-id>sub</nt:tp-id>
-            </nt:termination-point>
-          </nw:node>
-          <nw:node> <!-- /tf_static topic -->
-            <nw:node-id name="/camera/depth/image_rect_raw" />
-            <ros:ros-node-attributes>
-              <ros:ros-node-type>topic</ros:ros-node-type>
-              <ros:topic-type name="sensor_msgs/msg/Image" hz="30" bw="24.59MB/s"/>
-            </ros:ros-node-attributes>
-            <nt:termination-point>
-              <nt:tp-id>pub</nt:tp-id>
-            </nt:termination-point>
-            <nt:termination-point>
-              <nt:tp-id>sub</nt:tp-id>
-            </nt:termination-point>
-          </nw:node>
-      </xacro:macro>
+      <nw:network>
+        <nw:network-id>ros</nw:network-id>
+        <nw:network-types>
+          <ros:ros-node-graph/>
+        </nw:network-types>
+        <nw:supporting-network>
+          <nw:network-ref>${L2_network_id}</nw:network-ref>
+        </nw:supporting-network>
+        <nw:node> <!-- /camera/realsense2_camera ROS node -->
+          <nw:node-id>realsense2-camera</nw:node-id> <!--(node-name)-->
+          <ros:ros-node-attributes>
+            <ros:ros-node-type>node</ros:ros-node-type>
+          </ros:ros-node-attributes>
+          <nt:termination-point>
+            <nt:tp-id>pub</nt:tp-id>
+          </nt:termination-point>
+          <nt:termination-point>
+            <nt:tp-id>sub</nt:tp-id>
+          </nt:termination-point>
+        </nw:node>
+        <nw:node> <!-- /tf_static topic -->
+          <nw:node-id>/camera/color/image_raw</nw:node-id>
+          <ros:ros-node-attributes>
+            <ros:ros-node-type>topic</ros:ros-node-type>
+            <ros:topic-type>sensor_msgs/msg/Image</ros:topic-type>
+            <ros:hz>30</ros:hz>
+            <ros:bw>83.34MB/s</ros:bw>
+          </ros:ros-node-attributes>
+          <nt:termination-point>
+            <nt:tp-id>pub</nt:tp-id>
+          </nt:termination-point>
+          <nt:termination-point>
+            <nt:tp-id>sub</nt:tp-id>
+          </nt:termination-point>
+        </nw:node>
+        <nw:node> <!-- /tf_static topic -->
+          <nw:node-id>/camera/depth/image_rect_raw</nw:node-id>
+          <ros:ros-node-attributes>
+            <ros:ros-node-type>topic</ros:ros-node-type>
+            <ros:topic-type>sensor_msgs/msg/Image</ros:topic-type>
+            <ros:hz>30</ros:hz>
+            <ros:bw>24.59MB/s</ros:bw>
+          </ros:ros-node-attributes>
+          <nt:termination-point>
+            <nt:tp-id>pub</nt:tp-id>
+          </nt:termination-point>
+          <nt:termination-point>
+            <nt:tp-id>sub</nt:tp-id>
+          </nt:termination-point>
+        </nw:node>
+      </nw:network>
+      <nw:network>
+        <nw:network-id>${L2_network_id}</nw:network-id>
+        <nw:network-types>
+          <l2t:l2-topology/>
+        </nw:network-types>
+        <nw:supporting-network>
+          <nw:network-ref>${L1_network_id}</nw:network-ref>
+        </nw:supporting-network>
+        <nw:node>
+          <nw:node-id>${L2_id}</nw:node-id>
+          <nw:supporting-node>
+            <nw:network-ref>${L2_id}</nw:network-ref>
+            <nw:node-ref>${L1_id}</nw:node-ref>
+          </nw:supporting-node>
+          <xacro:usb30_L2 id="usb_1" supporting_network="${L1_network_id}" supporting_node="${L1_id}" supporting_tp="usb_1"/>
+        </nw:node>
+      </nw:network>
+      <nw:network>
+        <nw:network-id>${L1_network_id}</nw:network-id>
+        <nw:network-types>
+          <l1t:l1-topology/>
+        </nw:network-types>
+        <nw:node>
+          <nw:node-id>${L1_id}</nw:node-id>
+          <l1t:l1-node-attributes>
+            <l1t:device-type>camera</l1t:device-type>
+          </l1t:l1-node-attributes>
+          <xacro:usb30_L1 id="usb_1"/>
+        </nw:node>
+      </nw:network>
     </yang>
   </xacro:macro>

Commit message: Forgot the param list, added supporting node for ros, fixed a bug

File: realsense2_description/urdf/_d455.urdf.xacro (robot description, xacro)
@@ -29,5 +29,5 @@
   <xacro:include filename="$(find realsense2_description)/urdf/_materials.urdf.xacro" />
   <xacro:include filename="$(find realsense2_description)/urdf/_usb_plug.urdf.xacro" />
-  <xacro:macro name="sensor_d455" params="parent *origin name:=camera use_nominal_extrinsics:=false">
+  <xacro:macro name="sensor_d455" params="parent *origin name:=camera use_nominal_extrinsics:=false L2_network_id:=Data_Link L1_network_id:=Physical L2_id:=d455_Cam_L2 L1_id:=d455_Cam_L1 L3_network_id:=d455_Cam_ROS L3_id:=realsense2_camera">
     <xacro:arg name="add_plug" default="false" />
     <xacro:property name="M_PI" value="3.1415926535897931" />
@@ -200,4 +200,8 @@
             <ros:ros-node-type>node</ros:ros-node-type>
           </ros:ros-node-attributes>
+          <nw:supporting-node>
+            <nw:network-ref>${L2_network_id}</nw:network-ref>
+            <nw:node-ref>${L2_id}</nw:node-ref>
+          </nw:supporting-node>
           <nt:termination-point>
             <nt:tp-id>pub</nt:tp-id>
@@ -249,5 +253,5 @@
           <nw:node-id>${L2_id}</nw:node-id>
           <nw:supporting-node>
-            <nw:network-ref>${L2_id}</nw:network-ref>
+            <nw:network-ref>${L1_network_id}</nw:network-ref>
             <nw:node-ref>${L1_id}</nw:node-ref>
           </nw:supporting-node>

Commit message: ros layer removed

File: realsense2_description/urdf/_d455.urdf.xacro (robot description, xacro)
@@ -29,5 +29,5 @@
   <xacro:include filename="$(find realsense2_description)/urdf/_materials.urdf.xacro" />
   <xacro:include filename="$(find realsense2_description)/urdf/_usb_plug.urdf.xacro" />
-  <xacro:macro name="sensor_d455" params="parent *origin name:=camera use_nominal_extrinsics:=false L2_network_id:=Data_Link L1_network_id:=Physical L2_id:=d455_Cam_L2 L1_id:=d455_Cam_L1 L3_network_id:=d455_Cam_ROS L3_id:=realsense2_camera">
+  <xacro:macro name="sensor_d455" params="parent *origin name:=camera use_nominal_extrinsics:=false L2_network_id:=network_level L1_network_id:=device_level L2_id:=sensor_d455_L2 L1_id:=sensor_d455_L1">
     <xacro:arg name="add_plug" default="false" />
     <xacro:property name="M_PI" value="3.1415926535897931" />
@@ -188,59 +188,4 @@
     <yang>
       <nw:network>
-        <nw:network-id>ros</nw:network-id>
-        <nw:network-types>
-          <ros:ros-node-graph/>
-        </nw:network-types>
-        <nw:supporting-network>
-          <nw:network-ref>${L2_network_id}</nw:network-ref>
-        </nw:supporting-network>
-        <nw:node> <!-- /camera/realsense2_camera ROS node -->
-          <nw:node-id>realsense2-camera</nw:node-id> <!--(node-name)-->
-          <ros:ros-node-attributes>
-            <ros:ros-node-type>node</ros:ros-node-type>
-          </ros:ros-node-attributes>
-          <nw:supporting-node>
-            <nw:network-ref>${L2_network_id}</nw:network-ref>
-            <nw:node-ref>${L2_id}</nw:node-ref>
-          </nw:supporting-node>
-          <nt:termination-point>
-            <nt:tp-id>pub</nt:tp-id>
-          </nt:termination-point>
-          <nt:termination-point>
-            <nt:tp-id>sub</nt:tp-id>
-          </nt:termination-point>
-        </nw:node>
-        <nw:node> <!-- /tf_static topic -->
-          <nw:node-id>/camera/color/image_raw</nw:node-id>
-          <ros:ros-node-attributes>
-            <ros:ros-node-type>topic</ros:ros-node-type>
-            <ros:topic-type>sensor_msgs/msg/Image</ros:topic-type>
-            <ros:hz>30</ros:hz>
-            <ros:bw>83.34MB/s</ros:bw>
-          </ros:ros-node-attributes>
-          <nt:termination-point>
-            <nt:tp-id>pub</nt:tp-id>
-          </nt:termination-point>
-          <nt:termination-point>
-            <nt:tp-id>sub</nt:tp-id>
-          </nt:termination-point>
-        </nw:node>
-        <nw:node> <!-- /tf_static topic -->
-          <nw:node-id>/camera/depth/image_rect_raw</nw:node-id>
-          <ros:ros-node-attributes>
-            <ros:ros-node-type>topic</ros:ros-node-type>
-            <ros:topic-type>sensor_msgs/msg/Image</ros:topic-type>
-            <ros:hz>30</ros:hz>
-            <ros:bw>24.59MB/s</ros:bw>
-          </ros:ros-node-attributes>
-          <nt:termination-point>
-            <nt:tp-id>pub</nt:tp-id>
-          </nt:termination-point>
-          <nt:termination-point>
-            <nt:tp-id>sub</nt:tp-id>
-          </nt:termination-point>
-        </nw:node>
-      </nw:network>
-      <nw:network>
         <nw:network-id>${L2_network_id}</nw:network-id>
         <nw:network-types>

Commit message: yang content update

File: realsense2_description/urdf/_d455.urdf.xacro (robot description, xacro)
@@ -25,5 +25,5 @@
   <xacro:include filename="$(find realsense2_description)/urdf/_usb_plug.urdf.xacro" />
   <xacro:include filename="$(find interface_description)/urdf/usb-typec.urdf.xacro" />
-  <xacro:macro name="sensor_d455" params="parent *origin name:=camera use_nominal_extrinsics:=false L2_network_id:=sensor_d455_network_level L1_network_id:=sensor_d455_device_level L2_id:=sensor_d455_L2 L1_id:=sensor_d455_L1">
+  <xacro:macro name="sensor_d455" params="parent *origin name:=camera use_nominal_extrinsics:=false id:=0">
     <xacro:arg name="add_plug" default="false" />
     <xacro:property name="M_PI" value="3.1415926535897931" />
@@ -189,5 +189,5 @@
         <dl:device-type>camera</dl:device-type>
       </dl:device-layer-node-attributes>
-      <xacro:usb_typec parent="world" id="0" />
+      <xacro:usb_typec parent="${name}_link" prefix="${name}-${id}" id="0" origin_xyz="0.075 0.119 0.0199" origin_rpy="1.5707963 1.5707963 0"/>
     </node>
   </xacro:macro>

Commit message: unique naming

File: realsense2_description/urdf/_d455.urdf.xacro (robot description, xacro)
@@ -25,5 +25,5 @@
   <xacro:include filename="$(find realsense2_description)/urdf/_usb_plug.urdf.xacro" />
   <xacro:include filename="$(find interface_description)/urdf/usb-typec.urdf.xacro" />
-  <xacro:macro name="sensor_d455" params="parent *origin name:=camera use_nominal_extrinsics:=false id:=0">
+  <xacro:macro name="sensor_d455" params="parent *origin name:=d455 use_nominal_extrinsics:=false id:=0">
     <xacro:arg name="add_plug" default="false" />
     <xacro:property name="M_PI" value="3.1415926535897931" />
