Commit message: update namespaces

File: realsense2_description/urdf/_d435.urdf.xacro (robot description, xacro)
@@ -20,6 +20,5 @@
 -->
 <robot name="sensor_d435" xmlns:xacro="http://ros.org/wiki/xacro"
-       xmlns:nw="urn:template-network"
-       xmlns:nt="urn:network-topology"
+       xmlns:nw="urn:network"
        xmlns:l1t="urn:layer1"
        xmlns:l2t="urn:layer2">
@@ -28,5 +27,5 @@
   <xacro:include filename="$(find realsense2_description)/urdf/_usb_plug.urdf.xacro" />
   <xacro:include filename="$(find interface-description)/urdf/usb30.urdf.xacro" />
-  <xacro:macro name="sensor_d435" params="parent *origin name:=camera use_nominal_extrinsics:=false add_plug:=false use_mesh:=true L1_id L2_id L1_network_id L2_network_id">
+  <xacro:macro name="sensor_d435" params="parent *origin name:=camera use_nominal_extrinsics:=false add_plug:=false use_mesh:=true L1_id:=alma L2_id:=barack L1_network_id:=citrom L2_network_id:=dinnye">
     <xacro:property name="M_PI" value="3.1415926535897931" />
     <!-- The following values are approximate, and the camera node

Commit message: yang layer parameters updated

File: realsense2_description/urdf/_d435.urdf.xacro (robot description, xacro)
@@ -27,5 +27,5 @@
   <xacro:include filename="$(find realsense2_description)/urdf/_usb_plug.urdf.xacro" />
   <xacro:include filename="$(find interface-description)/urdf/usb30.urdf.xacro" />
-  <xacro:macro name="sensor_d435" params="parent *origin name:=camera use_nominal_extrinsics:=false add_plug:=false use_mesh:=true L1_id:=alma L2_id:=barack L1_network_id:=citrom L2_network_id:=dinnye">
+  <xacro:macro name="sensor_d435" params="parent *origin name:=camera use_nominal_extrinsics:=false add_plug:=false use_mesh:=true L1_id:=d435_L1 L2_id:=d435_L2 L1_network_id:=Physical L2_network_id:=Data_Link">
     <xacro:property name="M_PI" value="3.1415926535897931" />
     <!-- The following values are approximate, and the camera node

Commit message: p2668 conform layers

File: realsense2_description/urdf/_d435.urdf.xacro (robot description, xacro)
@@ -27,5 +27,5 @@
   <xacro:include filename="$(find realsense2_description)/urdf/_usb_plug.urdf.xacro" />
   <xacro:include filename="$(find interface-description)/urdf/usb30.urdf.xacro" />
-  <xacro:macro name="sensor_d435" params="parent *origin name:=camera use_nominal_extrinsics:=false add_plug:=false use_mesh:=true L1_id:=d435_L1 L2_id:=d435_L2 L1_network_id:=Physical L2_network_id:=Data_Link">
+  <xacro:macro name="sensor_d435" params="parent *origin name:=camera use_nominal_extrinsics:=false add_plug:=false use_mesh:=true L2_network_id:=network_level L1_network_id:=device_level L2_id:=sensor_d435_L2 L1_id:=sensor_d435_L1">
     <xacro:property name="M_PI" value="3.1415926535897931" />
     <!-- The following values are approximate, and the camera node

Commit message: attributes updated

File: realsense2_description/urdf/_d435.urdf.xacro (robot description, xacro)
@@ -19,11 +19,15 @@
 aluminum peripherial evaluation case.
 -->
-<robot name="sensor_d435" xmlns:xacro="http://ros.org/wiki/xacro"
-       xmlns:layer1="urn:ietf:params:xml:ns:yang:layer1">
+<robot name="sensor_d435"
+       xmlns:xacro="http://ros.org/wiki/xacro"
+       xmlns:layer1="urn:ietf:params:xml:ns:yang:layer1"
+       xmlns:layer2="urn:ietf:params:xml:ns:yang:layer2"
+       xmlns:robot-network="urn:ietf:params:xml:ns:yang:robot-network">
   <!-- Includes -->
   <xacro:include filename="$(find realsense2_description)/urdf/_materials.urdf.xacro" />
   <xacro:include filename="$(find realsense2_description)/urdf/_usb_plug.urdf.xacro" />
   <xacro:include filename="$(find interface-description)/urdf/usb30.urdf.xacro" />
-  <xacro:macro name="sensor_d435" params="parent *origin name:=camera use_nominal_extrinsics:=false add_plug:=false use_mesh:=true L2_network_id:=network_level L1_network_id:=device_level L2_id:=sensor_d435_L2 L1_id:=sensor_d435_L1">
+  <xacro:macro name="sensor_d435" params="parent *origin name:=camera use_nominal_extrinsics:=false add_plug:=false use_mesh:=true L2_network_id:=${name}_network_level L1_network_id:=${name}_device_level L2_id:=sensor_d435_L2 L1_id:=sensor_d435_L1">
+    <xacro:arg name="add_plug" default="false" />
     <xacro:property name="M_PI" value="3.1415926535897931" />
     <!-- The following values are approximate, and the camera node
@@ -45,5 +49,5 @@
     <!-- convenience precomputation to avoid clutter-->
     <xacro:property name="d435_mesh_x_offset" value="${d435_cam_mount_from_center_offset-d435_glass_to_front-d435_zero_depth_to_glass}"/>
-    <!-- The following offset is relative the the physical D435 camera peripherial
+    <!-- The following offset is relative to the physical D435 camera peripherial
   	camera tripod mount -->
     <xacro:property name="d435_cam_depth_px" value="${d435_cam_mount_from_center_offset}"/>
@@ -147,5 +151,5 @@
       <link name="${name}_color_optical_frame"/>
     </xacro:if>
-    <xacro:if value="${add_plug}">
+    <xacro:if value="${arg add_plug}">
       <xacro:usb_plug parent="${name}_link" name="${name}_usb_plug">
         <origin xyz="${d435_cam_mount_from_center_offset - 0.02095} ${-d435_cam_depth_py - 0.0353} 0" rpy="0 0 0"/>
@@ -154,6 +158,7 @@
     <yang>
       <!-- Realsense D435i L2 network topology -->
-      <network>
+      <robot-network:networks>
         <network-id>${L2_network_id}</network-id>
+        <layer2:l2-topology><element>template</element></layer2:l2-topology>
         <supporting-network>
           <network-ref>${L1_network_id}</network-ref>
@@ -168,16 +173,19 @@
           <xacro:usb30_L2 id="usb_1" supporting_network="${L1_network_id}" supporting_node="${L1_id}" supporting_tp="usb-typec_1"/>
         </node>
-      </network>
+      </robot-network:networks>
       <!-- Realsense D435i L1 network topology -->
-      <network>
+      <robot-network:networks>
         <network-id>${L1_network_id}</network-id>
+        <layer1:l1-topology><element>template</element></layer1:l1-topology>
         <node>
           <node-id>${L1_id}</node-id>
           <layer1:l1-node-attributes>
             <device-type>camera</device-type>
+            <phy-port-num>1</phy-port-num>
+            <wireless-access>0</wireless-access>
           </layer1:l1-node-attributes>
           <xacro:usb30_L1 id="usb_1" connector_type="usb_type-C" connector_format="female"/>
         </node>
-      </network>
+      </robot-network:networks>
     </yang>
   </xacro:macro>

File: realsense2_description/urdf/_d455.urdf.xacro (robot description, xacro)
@@ -21,9 +21,12 @@
 <robot name="sensor_d455"
        xmlns:xacro="http://ros.org/wiki/xacro"
-       xmlns:layer1="urn:ietf:params:xml:ns:yang:layer1">
+       xmlns:layer1="urn:ietf:params:xml:ns:yang:layer1"
+       xmlns:layer2="urn:ietf:params:xml:ns:yang:layer2"
+       xmlns:robot-network="urn:ietf:params:xml:ns:yang:robot-network">
   <!-- Includes -->
   <xacro:include filename="$(find realsense2_description)/urdf/_materials.urdf.xacro" />
   <xacro:include filename="$(find realsense2_description)/urdf/_usb_plug.urdf.xacro" />
-  <xacro:macro name="sensor_d455" params="parent *origin name:=camera use_nominal_extrinsics:=false L2_network_id:=network_level L1_network_id:=device_level L2_id:=sensor_d455_L2 L1_id:=sensor_d455_L1">
+  <xacro:include filename="$(find interface-description)/urdf/usb30.urdf.xacro" />
+  <xacro:macro name="sensor_d455" params="parent *origin name:=camera use_nominal_extrinsics:=false L2_network_id:=sensor_d455_network_level L1_network_id:=sensor_d455_device_level L2_id:=sensor_d455_L2 L1_id:=sensor_d455_L1">
     <xacro:arg name="add_plug" default="false" />
     <xacro:property name="M_PI" value="3.1415926535897931" />
@@ -183,6 +186,8 @@
     </xacro:if>
     <yang>
-      <network>
+      <!-- Realsense D455 L2 network topology -->
+      <robot-network:networks>
         <network-id>${L2_network_id}</network-id>
+        <layer2:l2-topology><element>template</element></layer2:l2-topology>
         <supporting-network>
           <network-ref>${L1_network_id}</network-ref>
@@ -195,17 +200,21 @@
             <node-ref>${L1_id}</node-ref>
           </supporting-node>
-          <xacro:usb30_L2 id="usb_1" supporting_network="${L1_network_id}" supporting_node="${L1_id}" supporting_tp="usb_1"/>
+          <xacro:usb30_L2 id="usb_1" supporting_network="${L1_network_id}" supporting_node="${L1_id}" supporting_tp="usb-typec_1"/>
         </node>
-      </network>
-      <network>
+      </robot-network:networks>
+      <!-- Realsense D455 L1 network topology -->
+      <robot-network:networks>
         <network-id>${L1_network_id}</network-id>
+        <layer1:l1-topology><element>template</element></layer1:l1-topology>
         <node>
           <node-id>${L1_id}</node-id>
           <layer1:l1-node-attributes>
             <device-type>camera</device-type>
+            <phy-port-num>2</phy-port-num>
+            <wireless-access>0</wireless-access>
           </layer1:l1-node-attributes>
           <xacro:usb30_L1 id="usb_1" connector_type="usb_type-C" connector_format="female"/>
         </node>
-      </network>
+      </robot-network:networks>
     </yang>
   </xacro:macro>

Commit message: yang ext update

File: realsense2_description/urdf/_d435.urdf.xacro (robot description, xacro)
@@ -24,6 +24,6 @@
   <xacro:include filename="$(find realsense2_description)/urdf/_materials.urdf.xacro" />
   <xacro:include filename="$(find realsense2_description)/urdf/_usb_plug.urdf.xacro" />
-  <xacro:include filename="$(find interface_description)/urdf/usb30.urdf.xacro" />
-  <xacro:macro name="sensor_d435" params="parent *origin name:=camera use_nominal_extrinsics:=false add_plug:=false use_mesh:=true L2_network_id:=${name}_network_level L1_network_id:=${name}_device_level L2_id:=sensor_d435_L2 L1_id:=sensor_d435_L1">
+  <xacro:include filename="$(find interface_description)/urdf/usb-typec.urdf.xacro" />
+  <xacro:macro name="sensor_d435" params="parent *origin name:=d435 use_nominal_extrinsics:=false add_plug:=false use_mesh:=true id:=0 ">
     <xacro:arg name="add_plug" default="false" />
     <xacro:property name="M_PI" value="3.1415926535897931" />
@@ -148,85 +148,19 @@
       <link name="${name}_color_optical_frame"/>
     </xacro:if>
-    <xacro:if value="${arg add_plug}">
+    <xacro:if value="${add_plug}">
       <xacro:usb_plug parent="${name}_link" name="${name}_usb_plug">
         <origin xyz="${d435_cam_mount_from_center_offset - 0.02095} ${-d435_cam_depth_py - 0.0353} 0" rpy="0 0 0"/>
       </xacro:usb_plug>
     </xacro:if>
-        <yang>
-            <!-- PoE switch network topology -->
-            <network>
-                <network-id>${L2_network_id}</network-id>
-                <supporting-network>
-                    <network-ref>${L1_network_id}</network-ref>
-                </supporting-network>
-                <node>
-                <node-id>${L2_id}</node-id>
-                <supporting-node>
-                    <network-ref>${L1_network_id}</network-ref>
-                    <node-ref>${L1_id}</node-ref>
-                </supporting-node>
-                <dl:device-layer-node-attributes xmlns:dl="urn:ietf:params:xml:ns:yang:device-layer">
-                    <dl:device-name>Intel RealSense D435</dl:device-name>
-                    <dl:device-type>camera</dl:device-type>
-                </dl:device-layer-node-attributes>
-                <nt:termination-point xmlns:nt="urn:ietf:params:xml:ns:yang:ietf-network-topology">
-                    <nt:tp-id>_0</nt:tp-id>
-                    <nt:supporting-termination-point>
-                        <nt:network-ref>${L2_id}</nt:network-ref>
-                        <nt:node-ref>${L1_id}</nt:node-ref>
-                        <nt:tp-ref>eth_0</nt:tp-ref>
-                    </nt:supporting-termination-point>
-                    <dl:device-layer-termination-point-attributes xmlns:dl="urn:ietf:params:xml:ns:yang:device-layer">
-                        <dl:port-name>port1</dl:port-name>
-                        <dl:port-type>rj45</dl:port-type>
-                    </dl:device-layer-termination-point-attributes>
-                    <nl:network-layer-termination-point-attributes xmlns:nl="urn:ietf:params:xml:ns:yang:network-layer">
-                        <nl:interface-name>intf1</nl:interface-name>
-                        <nl:interface-type>ethernet</nl:interface-type>
-                        <nl:interface-status>up</nl:interface-status>
-                        <nl:mac-address>00:1A:2B:3C:4D:5E</nl:mac-address>
-                    </nl:network-layer-termination-point-attributes>
-                </nt:termination-point>
-                <nl:network-layer-node-attributes xmlns:nl="urn:ietf:params:xml:ns:yang:network-layer">
-                    <nl:node-name>netNode1</nl:node-name>
-                    <nl:node-type>generic</nl:node-type>
-                </nl:network-layer-node-attributes>
-                </node>
-                <dl:device-layer-topology xmlns:dl="urn:ietf:params:xml:ns:yang:device-layer">
-                    <dl:element>element2</dl:element>
-                </dl:device-layer-topology>
-                <nt:link xmlns:nt="urn:ietf:params:xml:ns:yang:ietf-network-topology">
-                    <nt:link-id>link1</nt:link-id>
-                    <nt:source>
-                        <nt:source-node>node1</nt:source-node>
-                        <nt:source-tp>tp1</nt:source-tp>
-                    </nt:source>
-                    <nt:destination>
-                        <nt:dest-node>node2</nt:dest-node>
-                        <nt:dest-tp>tp2</nt:dest-tp>
-                    </nt:destination>
-                    <nt:supporting-link>
-                        <nt:network-ref>network2</nt:network-ref>
-                        <nt:link-ref>link2</nt:link-ref>
-                    </nt:supporting-link>
-                    <dl:device-layer-link-attributes xmlns:dl="urn:ietf:params:xml:ns:yang:device-layer">
-                        <dl:physical-link-name>physLink1</dl:physical-link-name>
-                        <dl:physical-link-type>cat5e</dl:physical-link-type>
-                    </dl:device-layer-link-attributes>
-                    <nl:network-layer-link-attributes xmlns:nl="urn:ietf:params:xml:ns:yang:network-layer">
-                        <nl:link-name>netLink1</nl:link-name>
-                        <nl:link-type>3gpp-5g-qos-flow</nl:link-type>
-                        <nl:_5qi>1</nl:_5qi>
-                        <nl:gfbr>50</nl:gfbr>
-                        <nl:mfbr>100</nl:mfbr>
-                        <nl:pdb>20</nl:pdb>
-                        <nl:per>0</nl:per>
-                    </nl:network-layer-link-attributes>
-                </nt:link>
-                <nl:network-layer-topology xmlns:nl="urn:ietf:params:xml:ns:yang:network-layer">
-                    <nl:element>element3</nl:element>
-                </nl:network-layer-topology>
-            </network>
-        </yang>
+    <!-- Intel RealSense D455 network topology -->
+    <node>
+      <node-id>${name}-${id}</node-id>
+      <dl:device-layer-node-attributes xmlns:dl="urn:ietf:params:xml:ns:yang:device-layer">
+        <dl:device-name>realsense-d435-camera</dl:device-name>
+        <dl:device-type>d435</dl:device-type>
+        <dl:weight>72</dl:weight>
+      </dl:device-layer-node-attributes>
+      <xacro:usb_typec parent="${name}_link" prefix="${name}-${id}" id="0" origin_xyz="-0.0167 -0.0435 0.0" origin_rpy="0 -1.57 1.57 "/>
+    </node>
   </xacro:macro>
 </robot>

Commit message: namespace fix

File: realsense2_description/urdf/_d435.urdf.xacro (robot description, xacro)
@@ -25,5 +25,6 @@
   <xacro:include filename="$(find realsense2_description)/urdf/_usb_plug.urdf.xacro" />
   <xacro:include filename="$(find interface_description)/urdf/usb-typec.urdf.xacro" />
-  <xacro:macro name="sensor_d435" params="parent *origin name:=d435 use_nominal_extrinsics:=false add_plug:=false use_mesh:=true id:=0 ">
+  <xacro:macro name="sensor_d435" params="parent *origin name:=d435 use_nominal_extrinsics:=false add_plug:=false use_mesh:=true id:=0 "
+    xmlns:nw="urn:ietf:params:xml:ns:yang:ietf-network">
     <xacro:arg name="add_plug" default="false" />
     <xacro:property name="M_PI" value="3.1415926535897931" />

File: realsense2_description/urdf/_d455.urdf.xacro (robot description, xacro)
@@ -25,5 +25,6 @@
   <xacro:include filename="$(find realsense2_description)/urdf/_usb_plug.urdf.xacro" />
   <xacro:include filename="$(find interface_description)/urdf/usb-typec.urdf.xacro" />
-  <xacro:macro name="sensor_d455" params="parent *origin name:=d455 use_nominal_extrinsics:=false id:=0">
+  <xacro:macro name="sensor_d455" params="parent *origin name:=d455 use_nominal_extrinsics:=false id:=0"
+    xmlns:nw="urn:ietf:params:xml:ns:yang:ietf-network">
     <xacro:arg name="add_plug" default="false" />
     <xacro:property name="M_PI" value="3.1415926535897931" />

Commit message: yang attributes fixed

File: realsense2_description/urdf/_d435.urdf.xacro (robot description, xacro)
@@ -154,13 +154,12 @@
       </xacro:usb_plug>
     </xacro:if>
-    <!-- Intel RealSense D455 network topology -->
+    <!-- Intel RealSense D435 network topology -->
     <node>
-      <node-id>${name}-${id}</node-id>
+      <node-id>${name}-${id}-node</node-id>
       <dl:device-layer-node-attributes xmlns:dl="urn:ietf:params:xml:ns:yang:device-layer">
         <dl:device-name>realsense-d435-camera</dl:device-name>
         <dl:device-type>d435</dl:device-type>
-        <dl:weight>72</dl:weight>
       </dl:device-layer-node-attributes>
-      <xacro:usb_typec parent="${name}_link" prefix="${name}-${id}" id="0" origin_xyz="-0.0167 -0.0435 0.0" origin_rpy="0 -1.57 1.57 "/>
+      <xacro:usb_typec parent="${name}-${id}-link" prefix="${name}-${id}" id="0" origin_xyz="-0.0167 -0.0435 0.0" origin_rpy="0 -1.57 1.57 "/>
     </node>
   </xacro:macro>

File: realsense2_description/urdf/_d455.urdf.xacro (robot description, xacro)
@@ -25,5 +25,5 @@
   <xacro:include filename="$(find realsense2_description)/urdf/_usb_plug.urdf.xacro" />
   <xacro:include filename="$(find interface_description)/urdf/usb-typec.urdf.xacro" />
-  <xacro:macro name="sensor_d455" params="parent *origin name:=d455 use_nominal_extrinsics:=false id:=0"
+  <xacro:macro name="sensor_d455" params="parent *origin name:=d455 use_nominal_extrinsics:=false add_plug:=false id:=0"
     xmlns:nw="urn:ietf:params:xml:ns:yang:ietf-network">
     <xacro:arg name="add_plug" default="false" />
@@ -62,7 +62,7 @@
       <origin xyz="${d455_mesh_x_offset} ${d455_cam_depth_py} ${d455_cam_depth_pz}" rpy="0 0 0"/>
       <parent link="${name}_bottom_screw_frame"/>
-      <child link="${name}_link" />
+      <child link="${name}-${id}-link" />
     </joint>
-    <link name="${name}_link">
+    <link name="${name}-${id}-link">
       <visual>
         <!-- the mesh origin is at front plate in between the two infrared camera axes -->
@@ -93,5 +93,5 @@
       <joint name="${name}_depth_joint" type="fixed">
         <origin xyz="0 0 0" rpy="0 0 0"/>
-        <parent link="${name}_link"/>
+        <parent link="${name}-${id}-link"/>
         <child link="${name}_depth_frame" />
       </joint>
@@ -106,5 +106,5 @@
       <joint name="${name}_infra1_joint" type="fixed">
         <origin xyz="0 ${d455_cam_depth_to_infra1_offset} 0" rpy="0 0 0" />
-        <parent link="${name}_link" />
+        <parent link="${name}-${id}-link" />
         <child link="${name}_infra1_frame" />
       </joint>
@@ -119,5 +119,5 @@
       <joint name="${name}_infra2_joint" type="fixed">
         <origin xyz="0 ${d455_cam_depth_to_infra2_offset} 0" rpy="0 0 0" />
-        <parent link="${name}_link" />
+        <parent link="${name}-${id}-link" />
         <child link="${name}_infra2_frame" />
       </joint>
@@ -132,5 +132,5 @@
       <joint name="${name}_color_joint" type="fixed">
         <origin xyz="0 ${d455_cam_depth_to_color_offset} 0" rpy="0 0 0" />
-        <parent link="${name}_link" />
+        <parent link="${name}-${id}-link" />
         <child link="${name}_color_frame" />
       </joint>
@@ -154,5 +154,5 @@
       <joint name="${name}_accel_joint" type="fixed">
         <origin xyz = "${d455_imu_px} ${d455_imu_py} ${d455_imu_pz}" rpy = "0 0 0" />
-        <parent link="${name}_link" />
+        <parent link="${name}-${id}-link" />
         <child link="${name}_accel_frame" />
       </joint>
@@ -164,5 +164,5 @@
       <joint name="${name}_gyro_joint" type="fixed">
         <origin xyz = "${d455_imu_px} ${d455_imu_py} ${d455_imu_pz}" rpy = "0 0 0" />
-        <parent link="${name}_link" />
+        <parent link="${name}-${id}-link" />
         <child link="${name}_gyro_frame" />
       </joint>
@@ -179,5 +179,5 @@
     </xacro:if>
     <xacro:if value="$(arg add_plug)">
-      <xacro:usb_plug parent="${name}_link" name="${name}_usb_plug">
+      <xacro:usb_plug parent="${name}-${id}-link" name="${name}_usb_plug">
         <origin xyz="${-0.00406-d455_cam_depth_px} ${-0.03701-d455_cam_depth_py} ${-d455_cam_depth_pz}" rpy="${M_PI/2} 0 0"/>
       </xacro:usb_plug>
@@ -185,11 +185,10 @@
     <!-- Intel RealSense D455 network topology -->
     <node>
-      <node-id>${name}-${id}</node-id>
+      <node-id>${name}-${id}-node</node-id>
       <dl:device-layer-node-attributes xmlns:dl="urn:ietf:params:xml:ns:yang:device-layer">
         <dl:device-name>realsense-d455-camera</dl:device-name>
         <dl:device-type>d455</dl:device-type>
-        <dl:weight>72</dl:weight>
       </dl:device-layer-node-attributes>
-      <xacro:usb_typec parent="${name}_link" prefix="${name}-${id}" id="0" origin_xyz="-0.015 -0.08 -0.005" origin_rpy="0 3.14 1.57 "/>
+      <xacro:usb_typec parent="${name}-${id}-link" prefix="${name}-${id}" id="0" origin_xyz="-0.015 -0.08 -0.005" origin_rpy="0 3.14 1.57 "/>
     </node>
   </xacro:macro>
